File: eagle/EmonMbed.brd (EAGLE design)
At the start: 100 x 80 mm, 127 parts, among them IC2 74HC595D, IC3 74HC595D, IC4 ADE7758RW, J1 CON_TERMINAL_BLOCK_02-5MM, J2 CON_TERMINAL_BLOCK_02-5MM, J3 CON_TERMINAL_BLOCK_02-5MM, J4 CON_TERMINAL_BLOCK_03-5MM, J7 CON_TERMINAL_BLOCK_02-5MM, Q1 25MHz, U1 STM32L152RBT6, U2 W5500, Y1 32.768kHz, Y2 32.768kHz

Commit message: new schematics and datasheet
Parts:
- added C37: 10uF, rcl:C/6032-28R
- added C38, C39, C40, C41, C42, C43, C44, C55, C56: 0.1uF, rcl:C0805
- added C45, C59: 10uF, rcl:153CLV-0605
- added C46, C60: 0.1uF, rcl:153CLV-0605
- added C47, C48, C49, C50, C51, C52, C53, C54: 100nF, rcl:C0603
- added D1, D2, D3, D4: 1N4001, diode:DO-214AC
- added IC6: REG1117, burr-brown:SOT223
- added IC7: 7805DT, linear:TO252
- added JP10, JP11: (no value), pinhead:1X08
- added JP12, JP13: (no value), pinhead:1X03
- added JP14: (no value), pinhead:1X02
- added L1: 150Mhz, rcl:POWER-CHOKE_WE-TPC
- added R41, R42: R120, resistor:R0603
- added R43: 10, SparkFun-Passives:0603-RES
- added SV1: (no value), con-lstb:MA08-1
- added T3, T9: (no value), transistor-neu-to92:SOT23-BEC
- added U$1, U$4: ADUM1402, adum140x:SO16W
- added U$3: ESP-07, esp-07:ESP-07
- added X2: (no value), con-ptr500:AK500/2-H
- C23, C24, C25, C26, C27, C28, C33, C34, C35, C36: device SparkFun-Passives:CAP-PTH-SMALL2 -> SparkFun-Passives:0603-CAP
- JP1: value ESP8266 -> Vsel; device pinhead:2X04 -> pinhead:1X03
- R26, R27, R28, R29, R30, R31, R32, R33, R34, R35, R36, R37, R38: device SparkFun-Passives:AXIAL-0.4 -> SparkFun-Passives:0603-RES
- R4: value 10k -> 10; device resistor:R0603 -> SparkFun-Passives:0603-RES
- moved R4 271.2 mm to (-96.0, -171.5)
- moved JP1 177.7 mm to (-110.0, -84.0)
- moved C21 116.9 mm to (4.50, 55.0), turned to 270 degrees
- moved R24 116.0 mm to (4.66, 51.2), turned to 270 degrees
- moved R22 112.0 mm to (14.4, 54.9), turned to 270 degrees
- moved C20 108.5 mm to (1.50, 55.0), turned to 270 degrees
- moved R21 108.4 mm to (17.0, 54.9), turned to 270 degrees
- moved R23 107.2 mm to (1.54, 51.2), turned to 90 degrees
- moved R25 86.3 mm to (11.9, 54.9), turned to 270 degrees
- moved C19 77.8 mm to (6.34, 55.0), turned to 90 degrees
- moved C18 75.6 mm to (9.35, 54.9), turned to 90 degrees
- moved R20 70.8 mm to (6.91, 68.8), flipped to the bottom, turned to 90 degrees
- moved R19 69.7 mm to (10.7, 68.8), flipped to the bottom, turned to 90 degrees
- moved U2 53.1 mm to (11.2, 41.4)
- moved IC1 8.60 mm to (-21.7, 6.97)
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Connections:
- removed net CS: JP2.7
- removed net PA0: U1.14
- removed net PA1: U1.15
- removed net PA10: U1.43
- removed net PA11: U1.44
- removed net PA12: U1.45
- removed net PA15: U1.50
- removed net PA4: U1.20
- removed net PA8: U1.41
- removed net PA9: U1.42
- removed net PB0: U1.26
- removed net PB1: U1.27
- removed net PB12: U1.33
- removed net PB13: U1.34
- removed net PB14: U1.35
- removed net PB15: U1.36
- removed net PB4: U1.56
- removed net PB5: U1.57
- removed net PB7: U1.59
- removed net PC10: U1.51
- removed net PC11: U1.52
- removed net PC12: U1.53
- removed net PC4: U1.24
- removed net PC5: U1.25
- removed net PC6: U1.37
- removed net PC7: U1.38
- removed net PC8: U1.39
- removed net PC9: U1.40
- removed net PD2: U1.54
- removed net SCLK: U2.33
- removed net SCSN: R8.1, U2.32
- removed net SDI(MOSI): JP2.4
- removed net SDO(MISO): JP2.1
- removed net SPI_CS: U1.58
- removed net SPI_MISO: U1.22
- removed net SPI_MOSI: U1.23
- removed net SPI_SCK: U1.21
- removed net TCK: U1.49
- removed net TMS: U1.46
- new net !CS: SV1.3
- new net ADE_CS: U$4.12, U1.45
- new net ADE_MISO: U$1.13, U1.49
- new net ADE_MOSI: U$1.11, U1.50
- new net ADE_SCK: U$1.12, U1.46
- new net APCF: U$1.14, U1.56
- new net AVADE: C44.1, IC4.4, R4.2
- new net DGND1: C51.2, C52.2
- new net ESP_GPIO0: JP13.2, U$3.GPIO0
- new net ESP_RX: JP14.1, U$3.URXD, U1.53
- new net ESP_TX: JP14.2, U$3.UTXD, U1.54
- new net ETH_CS: R8.1, U1.20, U2.32
- new net ETH_MISO: U1.22, U2.34
- new net ETH_MOSI: U1.23, U2.35
- new net ETH_SCK: U1.21, U2.33
- new net GESP: C54.2, JP12.2, JP13.3, U$3.GND, U$3.GPIO15
- new net GEXT: JP12.3
- new net IRQ: SV1.7, U$4.14, U1.58
- new net LCD_CS: JP2.7, U1.33
- new net LCD_MISO: JP2.1, U1.35
- new net LCD_MOSI: JP2.4, U1.36
- new net LCD_SCK: JP2.3, U1.34
- new net N$44: R41.2, T9.B
- new net N$45: R42.2, T3.B
- new net PWRKEY: R41.1
- new net VADE: C37.+, C38.1, C39.1, C40.1, C41.1, C42.1, C43.1, C60.+, D3.A, IC4.3, IC7.2, R4.1, U$1.1, U$1.10, U$1.16, U$1.7, U$4.1, U$4.10, U$4.16, U$4.7
- new net VARCF: U$4.13, U1.57
- new net VCC1: C51.1, C52.1
- new net VESP: C54.1, JP1.2, JP13.1, U$3.CH_PD, U$3.GPIO2, U$3.VCC
- new net VEXT: JP1.3
- new net VRAW: D1.A, D2.A, X2.1
- net !ADECS: now also U$4.5
- net ADEAPCF: now also U$1.3
- net ADEIN: now also U$1.6
- net ADEIRQ: now also U$4.4
- net ADEOUT: now also U$1.4
- net ADESCK: now also U$1.5
- net ADEVARCF: now also U$4.3
- net AGND: now also C44.2, C47.2, C48.2, C49.2, C50.2, C56.2, L1.1, R36.1, R37.1, R38.1; no longer R36.P$1, R37.P$1, R38.P$1
- net BOOT0: no longer R4.2
- net DGND: now also C37.-, C38.2, C39.2, C41.2, C43.2, C45.-, C46.-, C53.2, C55.2, C59.-, C60.-, IC6.1, IC7.3, JP12.1, L1.2, T3.E, T9.E, U$1.2, U$1.8, U$4.2, U$4.8, X2.2; no longer JP1.2, R4.1
- net GND: now also C40.2, C42.2, SV1.2, U$1.15, U$1.9, U$4.15, U$4.9
- net IAN: now also R29.1; no longer R29.P$1
- net IAP: now also R26.1; no longer R26.P$1
- net IBN: now also R30.1; no longer R30.P$1
- net IBP: now also R27.1; no longer R27.P$1
- net ICN: now also R31.1; no longer R31.P$1
- net ICP: now also R28.1; no longer R28.P$1
- net MISO: now also SV1.6; no longer U2.34
- net MOSI: now also SV1.4; no longer U2.35
- net N$10: now also R31.2; no longer R31.P$2
- net N$24: now also R28.2; no longer R28.P$2
- net N$27: now also R26.2; no longer R26.P$2
- net N$28: now also R29.2; no longer R29.P$2
- net N$30: now also R30.2; no longer R30.P$2
- net N$31: now also R27.2; no longer R27.P$2
- net N$35: now also R35.2; no longer R35.P$2
- net N$36: now also R32.2, R36.2; no longer R32.P$2, R36.P$2
- net N$37: now also R33.2, R37.2; no longer R33.P$2, R37.P$2
- net N$40: now also R34.2, R38.2; no longer R34.P$2, R38.P$2
- net Q1: now also JP10.1
- net Q10: now also JP11.2
- net Q11: now also JP11.3
- net Q12: now also JP11.4
- net Q13: now also JP11.5
- net Q14: now also JP11.6
- net Q15: now also JP11.7
- net Q16: now also JP11.8
- net Q2: now also JP10.2
- net Q3: now also JP10.3
- net Q4: now also JP10.4
- net Q5: now also JP10.5
- net Q6: now also JP10.6
- net Q7: now also JP10.7
- net Q8: now also JP10.8
- net Q9: now also JP11.1
- net RESET: now also R42.1
- net SCK: now also SV1.5; no longer JP2.3
- net SERIAL_RX: now also U1.43; no longer JP1.1, U1.17
- net SERIAL_TX: now also U1.42; no longer JP1.8, U1.16
- net SIM_PWRKEY: now also T9.C, U1.24
- net SIM_RESET: now also T3.C, U1.25
- net SIM_RX: now also U1.51
- net SIM_TX: now also U1.52
- net VAP: now also R32.1; no longer R32.P$1
- net VBP: now also R33.1; no longer R33.P$1
- net VCC: now also C47.1, C48.1, C49.1, C50.1, C56.1, R43.2, SV1.8; no longer IC4.4
- net VCP: now also R34.1; no longer R34.P$1
- net VDD: now also C46.+, C53.1, C55.1, D4.A, IC6.2, JP1.1, R43.1; no longer IC4.3, JP1.3, JP1.7
- net VIN: now also C45.+, C59.+, D1.C, D2.C, D3.C, D4.C, IC6.3, IC7.1
- net VN: now also R35.1; no longer R35.P$1
Routing:
- net VDD: track 0.00 -> 17.7 mm
- net N$23: track 0.00 -> 9.49 mm
- net N$22: track 0.00 -> 9.41 mm
- net TXP: track 0.00 -> 8.01 mm
- net TXN: track 0.00 -> 4.94 mm
- net N$29: track 0.00 -> 4.09 mm
- net N$26: track 0.00 -> 3.86 mm
- net N$11: track 0.00 -> 3.85 mm
- net DGND: track 0.00 -> 3.07 mm
- net AGND: track 0.00 -> 3.07 mm
- net N$12: track 0.00 -> 2.55 mm
- net VCC: track 0.00 -> 2.54 mm
- net RXN: track 0.00 -> 2.20 mm
- net RXP: track 0.00 -> 2.08 mm

Commit message: update schematic
Parts:
- removed JP10, JP11: (no value), pinhead:1X08
- added JP15, JP16: (no value), pinhead:2X05/90
Connections:
- net Q1: now also JP15.1; no longer JP10.1
- net Q10: now also JP16.2; no longer JP11.2
- net Q11: now also JP16.3; no longer JP11.3
- net Q12: now also JP16.4; no longer JP11.4
- net Q13: now also JP16.5; no longer JP11.5
- net Q14: now also JP16.6; no longer JP11.6
- net Q15: now also JP16.7; no longer JP11.7
- net Q16: now also JP16.8; no longer JP11.8
- net Q2: now also JP15.2; no longer JP10.2
- net Q3: now also JP15.3; no longer JP10.3
- net Q4: now also JP15.4; no longer JP10.4
- net Q5: now also JP15.5; no longer JP10.5
- net Q6: now also JP15.6; no longer JP10.6
- net Q7: now also JP15.7; no longer JP10.7
- net Q8: now also JP15.8; no longer JP10.8
- net Q9: now also JP16.1; no longer JP11.1
Changed lines of the file:
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@@
 <element name="R40" library="resistor" package="R0603" value="10k" x="-113.03" y="-24.13"/>
 <element name="JP9" library="pinhead" package="1X04" value="USART" x="-107.95" y="-30.48"/>
-<element name="JP10" library="pinhead" package="1X08" value="" x="-103.5" y="-38"/>
-<element name="JP11" library="pinhead" package="1X08" value="" x="-103.5" y="-44.5"/>
 <element name="U$3" library="esp-07" package="ESP-07" value="ESP-07" x="-103.5" y="-73.5"/>
 <element name="JP1" library="pinhead" package="1X03" value="Vsel" x="-110" y="-84"/>
@@
 <element name="C45" library="rcl" package="153CLV-0605" value="10uF" x="-172" y="-276"/>
 <element name="C46" library="rcl" package="153CLV-0605" value="0.1uF" x="-182" y="-276"/>
+<element name="JP15" library="pinhead" package="2X05/90" value="" x="-177" y="-291"/>
+<element name="JP16" library="pinhead" package="2X05/90" value="" x="-177" y="-307"/>
 </elements>
 <signals>
@@
 <signal name="Q8">
 <contactref element="IC2" pad="7"/>
-<contactref element="JP10" pad="8"/>
-<wire x1="-79.375" y1="70.5866" x2="-94.61" y2="-38" width="0" layer="19" extent="1-1"/>
+<contactref element="JP15" pad="8"/>
+<wire x1="-79.375" y1="70.5866" x2="-174.46" y2="-294.81" width="0" layer="19" extent="1-1"/>
 </signal>
 <signal name="Q7">
 <contactref element="IC2" pad="6"/>
-<contactref element="JP10" pad="7"/>
-<wire x1="-80.645" y1="70.5866" x2="-97.15" y2="-38" width="0" layer="19" extent="1-1"/>
+<contactref element="JP15" pad="7"/>
+<wire x1="-80.645" y1="70.5866" x2="-174.46" y2="-297.35" width="0" layer="19" extent="1-1"/>
 </signal>
 <signal name="Q6">
 <contactref element="IC2" pad="5"/>
-<contactref element="JP10" pad="6"/>
-<wire x1="-81.915" y1="70.5866" x2="-99.69" y2="-38" width="0" layer="19" extent="1-1"/>
+<contactref element="JP15" pad="6"/>
+<wire x1="-81.915" y1="70.5866" x2="-177" y2="-294.81" width="0" layer="19" extent="1-1"/>
 </signal>
 <signal name="Q5">
 <contactref element="IC2" pad="4"/>
-<contactref element="JP10" pad="5"/>
-<wire x1="-83.185" y1="70.5866" x2="-102.23" y2="-38" width="0" layer="19" extent="1-1"/>
+<contactref element="JP15" pad="5"/>
+<wire x1="-83.185" y1="70.5866" x2="-177" y2="-297.35" width="0" layer="19" extent="1-1"/>
 </signal>
 <signal name="Q4">
 <contactref element="IC2" pad="3"/>
-<contactref element="JP10" pad="4"/>
-<wire x1="-84.455" y1="70.5866" x2="-104.77" y2="-38" width="0" layer="19" extent="1-1"/>
+<contactref element="JP15" pad="4"/>
+<wire x1="-84.455" y1="70.5866" x2="-179.54" y2="-294.81" width="0" layer="19" extent="1-1"/>
 </signal>
 <signal name="Q3">
 <contactref element="IC2" pad="2"/>
-<contactref element="JP10" pad="3"/>
-<wire x1="-85.725" y1="70.5866" x2="-107.31" y2="-38" width="0" layer="19" extent="1-1"/>
+<contactref element="JP15" pad="3"/>
+<wire x1="-85.725" y1="70.5866" x2="-179.54" y2="-297.35" width="0" layer="19" extent="1-1"/>
 </signal>
 <signal name="Q2">
 <contactref element="IC2" pad="1"/>
-<contactref element="JP10" pad="2"/>
-<wire x1="-86.995" y1="70.5866" x2="-109.85" y2="-38" width="0" layer="19" extent="1-1"/>
+<contactref element="JP15" pad="2"/>
+<wire x1="-86.995" y1="70.5866" x2="-182.08" y2="-294.81" width="0" layer="19" extent="1-1"/>
 </signal>
 <signal name="Q1">
 <contactref element="IC2" pad="15"/>
-<contactref element="JP10" pad="1"/>
-<wire x1="-85.725" y1="76.7334" x2="-112.39" y2="-38" width="0" layer="19" extent="1-1"/>
+<contactref element="JP15" pad="1"/>
+<wire x1="-85.725" y1="76.7334" x2="-182.08" y2="-297.35" width="0" layer="19" extent="1-1"/>
 </signal>
 <signal name="Q16">
 <contactref element="IC3" pad="7"/>
-<contactref element="JP11" pad="8"/>
-<wire x1="-93.345" y1="70.5866" x2="-94.61" y2="-44.5" width="0" layer="19" extent="1-1"/>
+<contactref element="JP16" pad="8"/>
+<wire x1="-93.345" y1="70.5866" x2="-174.46" y2="-310.81" width="0" layer="19" extent="1-1"/>
 </signal>
 <signal name="Q15">
 <contactref element="IC3" pad="6"/>
-<contactref element="JP11" pad="7"/>
-<wire x1="-94.615" y1="70.5866" x2="-97.15" y2="-44.5" width="0" layer="19" extent="1-1"/>
+<contactref element="JP16" pad="7"/>
+<wire x1="-94.615" y1="70.5866" x2="-174.46" y2="-313.35" width="0" layer="19" extent="1-1"/>
 </signal>
 <signal name="Q14">
 <contactref element="IC3" pad="5"/>
-<contactref element="JP11" pad="6"/>
-<wire x1="-95.885" y1="70.5866" x2="-99.69" y2="-44.5" width="0" layer="19" extent="1-1"/>
+<contactref element="JP16" pad="6"/>
+<wire x1="-95.885" y1="70.5866" x2="-177" y2="-310.81" width="0" layer="19" extent="1-1"/>
 </signal>
 <signal name="Q13">
 <contactref element="IC3" pad="4"/>
-<contactref element="JP11" pad="5"/>
-<wire x1="-97.155" y1="70.5866" x2="-102.23" y2="-44.5" width="0" layer="19" extent="1-1"/>
+<contactref element="JP16" pad="5"/>
+<wire x1="-97.155" y1="70.5866" x2="-177" y2="-313.35" width="0" layer="19" extent="1-1"/>
 </signal>
 <signal name="Q12">
 <contactref element="IC3" pad="3"/>
-<contactref element="JP11" pad="4"/>
-<wire x1="-98.425" y1="70.5866" x2="-104.77" y2="-44.5" width="0" layer="19" extent="1-1"/>
+<contactref element="JP16" pad="4"/>
+<wire x1="-98.425" y1="70.5866" x2="-179.54" y2="-310.81" width="0" layer="19" extent="1-1"/>
 </signal>
 <signal name="Q11">
 <contactref element="IC3" pad="2"/>
-<contactref element="JP11" pad="3"/>
-<wire x1="-99.695" y1="70.5866" x2="-107.31" y2="-44.5" width="0" layer="19" extent="1-1"/>
+<contactref element="JP16" pad="3"/>
+<wire x1="-99.695" y1="70.5866" x2="-179.54" y2="-313.35" width="0" layer="19" extent="1-1"/>
 </signal>
 <signal name="Q10">
 <contactref element="IC3" pad="1"/>
-<contactref element="JP11" pad="2"/>
-<wire x1="-100.965" y1="70.5866" x2="-109.85" y2="-44.5" width="0" layer="19" extent="1-1"/>
+<contactref element="JP16" pad="2"/>
+<wire x1="-100.965" y1="70.5866" x2="-182.08" y2="-310.81" width="0" layer="19" extent="1-1"/>
 </signal>
 <signal name="Q9">
 <contactref element="IC3" pad="15"/>
-<contactref element="JP11" pad="1"/>
-<wire x1="-99.695" y1="76.7334" x2="-112.39" y2="-44.5" width="0" layer="19" extent="1-1"/>
+<contactref element="JP16" pad="1"/>
+<wire x1="-99.695" y1="76.7334" x2="-182.08" y2="-313.35" width="0" layer="19" extent="1-1"/>
 </signal>
 <signal name="QS">

Commit message: Updated Final Schematics
Parts:
- removed C1, C13, C47, C48, C49, C5, C50, C51, C52, C53, C54, C6, C7, C8, C9: 100nF, rcl:C0603
- removed C10, C11: 20pF, rcl:C0603
- removed C10-4U7, C11-22P, C9-100N: (no value), rcl:C0603
- removed C12: 1uF, rcl:C0603
- removed C14, C2: 4.7uF, rcl:C0603
- removed C15, C19: 10nF, rcl:C0603
- removed C16, C17: 18pF, rcl:C0603
- removed C18: 22nF, rcl:C0603
- removed C20, C21: 6.8nF, rcl:C0603
- removed C22: 1nF, rcl:C0603
- removed C23, C24, C25, C26, C27, C28, C33, C34, C35, C36: 33nF, SparkFun-Passives:0603-CAP
- removed C29: 0.1uF, rcl:C0805K
- removed C3, C4: 4.3pF, rcl:C0603
- removed C30: 10uF, rcl:C0805K
- removed C31, C32: 22pF, rcl:C0805K
- removed C37: 10uF, rcl:C/6032-28R
- removed C38, C39, C40, C41, C42, C43, C44, C55, C56: 0.1uF, rcl:C0805
- removed C45, C59: 10uF, rcl:153CLV-0605
- removed C46, C60: 0.1uF, rcl:153CLV-0605
- removed C7-100U: 100uF, rcl:153CLV-0605
- removed C8-100U: (no value), rcl:153CLV-0605
- removed CN1: (no value), microbuilder:RJ45_PULSEJACK
- removed CSIM_100N, CSIM_22P: (no value), rcl:C0603K
- removed D1, D2, D3, D4: 1N4001, diode:DO-214AC
- removed IC6: REG1117, burr-brown:SOT223
- removed IC7: 7805DT, linear:TO252
- removed J1, J2, J3, J7: CON_TERMINAL_BLOCK_02-5MM, dp_devices:TERMINAL_BLOCK_2P_5
- removed J4: CON_TERMINAL_BLOCK_03-5MM, dp_devices:TERMINAL_BLOCK_3P_5
- removed JP1: Vsel, pinhead:1X03
- removed JP12, JP13: (no value), pinhead:1X03
- removed JP14: (no value), pinhead:1X02
- removed JP15, JP16: (no value), pinhead:2X05/90
- removed JP2: TFT LCD ILI9341, pinhead:1X09
- removed JP3: SD CARD TFT LCD, pinhead:1X04
- removed JP4, JP5, JP6: (no value), jumper:JP1
- removed JP7: BOOT0, pinhead:1X03
- removed JP8: BOOT1, pinhead:1X03
- removed JP9: USART, pinhead:1X04
- removed L1: 150Mhz, rcl:POWER-CHOKE_WE-TPC
- removed L1600R: BLM15HB121SN1, inductors:0402
- removed LED1, LED2: (no value), microbuilder:CHIPLED_0805_NOOUTLINE
- removed Q1: 25MHz, special:QS
- removed R1, R3: 100R, resistor:R0603
- removed R10, R11, R12, R13, R14, R15, R16, R17, R18, R39, R40, R6, R7, R8: 10k, resistor:R0603
- removed R10-22, R11-22, R20-1K, R23-1K, R25-10K, R26-1K, R27-1K, R28-10K, R9-22: (no value), rcl:R0603
- removed R19, R20: 330, resistor:R0603
- removed R2: 4k7, resistor:R0603
- removed R21, R22, R23, R24: 49R9, resistor:R0603
- removed R25: 10R, resistor:R0603
- removed R26, R27, R28, R29, R30, R31, R35, R36, R37, R38: 1K, SparkFun-Passives:0603-RES
- removed R32, R33, R34: 1M, SparkFun-Passives:0603-RES
- removed R4, R43: 10, SparkFun-Passives:0603-RES
- removed R41, R42: R120, resistor:R0603
- removed R5: 12.4k, resistor:R0603
- removed R9: 1M, resistor:R0603
- removed S1, S2: SWITCH-MOMENTARY-2PTH, SparkFun-Electromechanical:TACTILE-PTH
- removed SV1: (no value), con-lstb:MA08-1
- removed T1, T2: (no value), transistor:SOT23-BEC
- removed T3, T9: (no value), transistor-neu-to92:SOT23-BEC
- removed U$1, U$4: ADUM1402, adum140x:SO16W
- removed U$2: SIMHOLDER3, SparkFun:SIMHOLDER3
- removed U$3: ESP-07, esp-07:ESP-07
- removed U$6: DCDCMODULE_SMALL, bontor:DCDCMODULE-SMALL
- removed U1: STM32L152RBT6, ST Microelctronics_By_element14_Batch_1:QFP50P1200X1200X160-64N
- removed X1: (no value), microbuilder:SMA90_DIP
- removed X2: (no value), con-ptr500:AK500/2-H
- removed Y1, Y2: 32.768kHz, SparkFun-FreqCtrl:TC26H
- removed Y3: (no value), SparkFun-FreqCtrl:HC49US
- added ADE-7, ADE-R10, ADE-R4: 33R, SparkFun-Passives:0603-RES
- added ADE-C1, ADE-C2, ADE-C3, ADE-C4, ADE-C5, ADE-C6, ADE-C7, ADE-C8: 33nF, SparkFun-Passives:0603-CAP
- added ADE-C10: 10uF, rcl:C0805K
- added ADE-C11, ADE-C12: 22pF, rcl:C0805K
- added ADE-C13: 10uF, rcl:C/6032-28R
- added ADE-C14, SYS-C1, SYS-C2, SYS-C3, SYS-C4: 0.1uF, rcl:C0805
- added ADE-C9: 0.1uF, rcl:C0805K
- added ADE-R1: 81K, SparkFun-Passives:0603-RES
- added ADE-R12, ADE-R2, ADE-R3, ADE-R5, ADE-R6, ADE-R8, ADE-R9, ADER-11: 1K, SparkFun-Passives:0603-RES
- added ADE-XTAL: 10MHz, SparkFun-FreqCtrl:HC49US
- added CT1, CT2, CT3: 100A, microbuilder:STX3100
- added DCDC-3.5V: DCDCMODULE_SMALL, bontor:DCDCMODULE-SMALL
- added ESP-C1, SIM900-C5, STM-C10, STM-C11, STM-C12, STM-C13, STM-C7, STM-C8, STM-C9, W5500-C10, W5500-C11, W5500-C5, W5500-C6, W5500-C7, W5500-C8, W5500-C9: 100nF, rcl:C0603
- added ESP-GND, LCD_SD: (no value), pinhead:1X04
- added ESP-GPIO0: (no value), pinhead:1X03
- added ESP-USART: (no value), pinhead:1X02
- added ESP-VDD: Vsel, pinhead:1X04
- added ESP8266: ESP-07, esp-07:ESP-07
- added ETH-C1: 22nF, rcl:C0603
- added ETH-C2, ETH-C4: 6.8nF, rcl:C0603
- added ETH-C3, W5500-C4: 10nF, rcl:C0603
- added ETH-R1, ETH-R2, ETH-R6, ETH-R7: 49R9, resistor:R0603
- added ETH-R3: 10R, resistor:R0603
- added ETH-R4, ETH-R5: 330, resistor:R0603
- added ETHERNET: (no value), microbuilder:RJ45_PULSEJACK
- added J5: POWER_JACKPTH, SparkFun-Connectors:POWER_JACK_PTH
- added LCD-R1: 680R, SparkFun-Passives:0603-RES
- added LCD_ILI9341: (no value), pinhead:1X09
- added SIM900-ANT: (no value), microbuilder:SMA90_DIP
- added SIM900-C1, SIM900-C2, SIM900-C3: 100uF, rcl:153CLV-0605
- added SIM900-C4: 4u7, rcl:C0603
- added SIM900-C6: 22pF, rcl:C0603
- added SIM900-LED1, SIM900-LED2: (no value), microbuilder:CHIPLED_0805_NOOUTLINE
- added SIM900-R1, SIM900-R2, SIM900-R3: 22R, rcl:R0603
- added SIM900-R10, SIM900-R11: 120R, resistor:R0603
- added SIM900-R4, SIM900-R7: 680R, rcl:R0603
- added SIM900-R5, SIM900-R8: 1K, rcl:R0603
- added SIM900-R6, SIM900-R9: 10K, rcl:R0603
- added SIM900-T1, SIM900-T2: (no value), transistor:SOT23-BEC
- added SIM900-T3, SIM900-T4: (no value), transistor-neu-to92:SOT23-BEC
- added SIM_C1: 100nF, rcl:C0603K
- added SIM_C2: 22pF, rcl:C0603K
- added SIM_HOLDER: SIMHOLDER3, SparkFun:SIMHOLDER3
- added SR_OUT1, SR_OUT2: (no value), pinhead:2X04/90
- added STM-C1: 1uF, rcl:C0603
- added STM-C2, STM-C3: 20pF, rcl:C0603
- added STM-C5, STM-C6: 4.3pF, rcl:C0603
- added STM-L1: BLM15HB121SN1, inductors:0402
- added STM-R1: 4k7, resistor:R0603
- added STM-R2, STM-R3: 100R, resistor:R0603
- added STM-S1, STM-S2: SWITCH-MOMENTARY-2PTH, SparkFun-Electromechanical:TACTILE-PTH
- added STM-USART: USART, pinhead:1X05
- added STM-XTAL1, STM-XTAL2: 32.768kHz, SparkFun-FreqCtrl:TC26H
- added STM_CHIP: STM32F103RBT6, ST Microelctronics_By_element14_Batch_1:QFP50P1200X1200X160-64N
- added SYS-L1: 150Mhz, rcl:POWER-CHOKE_WE-TPC
- added SYS-R1, SYS-R2: 10R, SparkFun-Passives:0603-RES
- added VAC_IN: 9V, SparkFun-Connectors:POWER_JACK_PTH
- added W5500-C1, W5500-C2: 18pF, rcl:C0603
- added W5500-C3: 4.7uF, rcl:C0603
- added W5500-HD1: BOOT0, pinhead:1X03
- added W5500-HD2: BOOT1, pinhead:1X03
- added W5500-R1, W5500-R11, W5500-R12, W5500-R13, W5500-R2, W5500-R3, W5500-R4, W5500-R5, W5500-R6, W5500-R7, W5500-R8, W5500-R9: 10k, resistor:R0603
- added W5500-R10: 1M, resistor:R0603
- added W5500-XTAL: 25MHz, special:QS
- IC1: value (none) -> SIM900
- moved IC1 186.9 mm to (-166.7, 125.0)
- moved IC2 161.2 mm to (32.5, -39.3)
- moved IC3 157.4 mm to (12.5, -39.8)
- moved IC4 150.2 mm to (-164.6, 16.2)
- moved U2 54.1 mm to (65.0, 47.0)
Connections:
- removed net !ADECS: IC4.21, U$4.5
- removed net !CS: SV1.3
- removed net ADEAPCF: IC4.1, U$1.3
- removed net ADEIN: IC4.22, U$1.6
- removed net ADEIRQ: IC4.18, U$4.4
- removed net ADEOUT: IC4.24, U$1.4
- removed net ADESCK: IC4.23, U$1.5
- removed net ADEVARCF: IC4.17, U$4.3
- removed net APCF: U$1.14, U1.56
- removed net AVADE: C44.1, IC4.4, R4.2
- removed net D/C: JP2.5
- removed net DGND1: C51.2, C52.2
- removed net DS_OE: IC2.13, IC3.13
- removed net EXRES1: R5.2, U2.10
- removed net I2C_SCL: U1.61
- removed net I2C_SDA: U1.62
- removed net IAN: J1.1, R29.1
- removed net IAP: J1.2, R26.1
- removed net IBP: J2.2, R27.1
- removed net ICP: J3.2, JP5.2, R28.1
- removed net INTN: R7.1, U2.36
- removed net IRQ: SV1.7, U$4.14, U1.58
- removed net LED: JP2.2
- removed net MISO: SV1.6
- removed net MOSI: SV1.4
- removed net N$10: C28.1, IC4.10, R31.2
- removed net PB10: U1.29
- removed net PB11: C2.1, U1.30
- removed net PWRKEY: R41.1
- removed net RESET: JP2.6, R42.1
- removed net RSTN: R13.1, U2.37
- removed net SCK: SV1.5
- removed net SD_MISO: JP3.3
- removed net SD_MOSI: JP3.2
- removed net SD_SCK: JP3.4
- removed net SHCP: IC2.11, IC3.11, U1.10
- removed net STCP: IC2.12, IC3.12, U1.9
- removed net VADE: C37.+, C38.1, C39.1, C40.1, C41.1, C42.1, C43.1, C60.+, D3.A, IC4.3, IC7.2, R4.1, U$1.1, U$1.10, U$1.16, U$1.7, U$4.1, U$4.10, U$4.16, U$4.7
- removed net VAP: J4.1, R32.1
- removed net VARCF: U$4.13, U1.57
- removed net VBP: J4.2, R33.1
- removed net VCC1: C51.1, C52.1
- removed net VCP: J4.3, JP6.2, R34.1
- removed net VIN: C45.+, C59.+, D1.C, D2.C, D3.C, D4.C, IC6.3, IC7.1, U$6.INP#1, U$6.INP#2
- removed net VN: J7.1, J7.2, R35.1
- removed net VRAW: D1.A, D2.A, X2.1
- removed net VSIM: C7-100U.+, C8-100U.+, IC1.P$55, IC1.P$56, IC1.P$57, U$6.OUTP#1, U$6.OUTP#2
- new net ADE_APCF: IC4.1, STM_CHIP.57
- new net ADE_IRQ: IC4.18, STM_CHIP.59
- new net ADE_VARCF: IC4.17, STM_CHIP.58
- new net AVDD: IC4.4, SYS-C2.1, SYS-R1.2
- new net ETH_RSTN: STM_CHIP.37, U2.37, W5500-R9.1
- new net LCD_D/C: LCD_ILI9341.5, STM_CHIP.24
- new net LCD_LED: LCD-R1.1, LCD_ILI9341.2
- new net LCD_RESET: LCD_ILI9341.6, STM_CHIP.25
- new net N$39: ADE-R4.2, ADE-R5.1, CT1.1
- new net N$47: ADE-R4.1, ADE-R6.1, CT1.5
- new net N$48: ADE-R10.2, ADER-11.1, CT3.1
- new net N$51: ADE-R3.1, VAC_IN.GND, VAC_IN.GNDBREAK
- new net SIM900_PWRKEY: IC1.P$1, SIM900-T3.C
- new net SIM900_RESET: IC1.P$16, SIM900-T4.C
- new net SR_SHCP: IC2.11, IC3.11, STM_CHIP.9
- new net SR_STCP: IC2.12, IC3.12, STM_CHIP.10
- net +5V: now also ADE-C13.+, ADE-C14.1, DCDC-3.5V.INP#1, DCDC-3.5V.INP#2, IC4.3, J5.PWR, SYS-C1.1, SYS-R1.1; no longer R20-1K.2, R26-1K.2
- net ACTLED: now also ETH-R4.1; no longer R19.1
- net ADE_CS: now also IC4.21, STM_CHIP.50; no longer U$4.12, U1.45
- net ADE_MISO: now also IC4.24, STM_CHIP.45; no longer U$1.13, U1.49
- net ADE_MOSI: now also IC4.22, STM_CHIP.46; no longer U$1.11, U1.50
- net ADE_SCK: now also IC4.23, STM_CHIP.49; no longer U$1.12, U1.46
- net AGND: now also ADE-C1.2, ADE-C10.2, ADE-C2.2, ADE-C3.2, ADE-C4.2, ADE-C5.2, ADE-C6.2, ADE-C7.2, ADE-C8.2, ADE-C9.2, ADE-R2.1, ETHERNET.4, ETHERNET.5, STM-C9.2, STM_CHIP.12, SYS-C2.2, SYS-C4.2, SYS-L1.1, W5500-C10.2, W5500-C11.2, W5500-C3.2, W5500-C4.2, W5500-C6.2, W5500-C7.2, W5500-C8.2, W5500-C9.2, W5500-R11.1; no longer C1.2, C14.2, C15.2, C22.1, C23.2, C24.2, C25.2, C26.2, C27.2, C28.2, C29.2, C30.2, C33.2, C34.2, C35.2, C36.2, C44.2, C47.2, C48.2, C49.2, C50.2, C56.2, CN1.4, CN1.5, JP4.1, JP5.1, JP6.1, L1.1, R36.1, R37.1, R38.1, R6.1, U1.12
- net BOOT0: now also STM_CHIP.60, W5500-R13.1; no longer R39.1, U1.60
- net BOOT1: now also STM_CHIP.28, W5500-R12.1; no longer R40.1, U1.28
- net DGND: now also ADE-C11.2, ADE-C12.2, ADE-C13.-, ADE-C14.2, DCDC-3.5V.INM#1, DCDC-3.5V.INM#2, DCDC-3.5V.OUTM#1, DCDC-3.5V.OUTM#2, ESP-GND.1, ETH-C1.1, ETH-C3.1, IC2.13, IC2.8, IC3.13, IC3.8, J5.GND, J5.GNDBREAK, LCD_ILI9341.8, SIM900-ANT.GND1, SIM900-ANT.GND2, SIM900-ANT.GND3, SIM900-ANT.GND4, SIM900-C1.-, SIM900-C2.-, SIM900-C3.-, SIM900-C4.2, SIM900-C5.2, SIM900-C6.2, SIM900-R6.2, SIM900-R9.2, SIM900-T1.E, SIM900-T2.E, SIM900-T3.E, SIM900-T4.E, SIM_C1.1, SIM_C2.1, SIM_HOLDER.6, STM-C1.1, STM-C10.2, STM-C11.2, STM-C12.2, STM-C13.2, STM-C2.1, STM-C3.2, STM-C5.1, STM-C6.2, STM-R2.1, STM-R3.1, STM-S1.1, STM-S2.1, STM-USART.5, STM_CHIP.18, STM_CHIP.31, STM_CHIP.47, STM_CHIP.63, SYS-C1.2, SYS-C3.2, SYS-L1.2, W5500-C1.2, W5500-C2.2, W5500-C5.2, W5500-HD1.3, W5500-HD2.3, W5500-R4.2, W5500-R5.2, W5500-R6.2, W5500-R7.2, W5500-R8.2; no longer C10-4U7.2, C10.2, C11-22P.2, C11.1, C12.1, C16.2, C17.2, C18.1, C19.1, C2.2, C22.2, C3.2, C31.2, C32.2, C37.-, C38.2, C39.2, C4.1, C41.2, C43.2, C45.-, C46.-, C53.2, C55.2, C59.-, C6.2, C60.-, C7-100U.-, C7.2, C8-100U.-, C8.2, C9-100N.2, C9.2, CSIM_100N.1, CSIM_22P.1, IC6.1, IC7.3, JP12.1, JP7.3, JP8.3, JP9.4, L1.2, R1.1, R14.2, R15.2, R16.2, R17.2, R18.2, R3.1, R5.1, S1.1, S2.1, T3.E, T9.E, U$1.2, U$1.8, U$2.6, U$4.2, U$4.8, U$6.INM#1, U$6.INM#2, U$6.OUTM#1, U$6.OUTM#2, U1.18, U1.31, U1.47, U1.63, X1.GND1, X1.GND2, X1.GND3, X1.GND4, X2.2
- net ESP_GPIO0: now also ESP-GPIO0.2, ESP8266.GPIO0; no longer JP13.2, U$3.GPIO0
- net ESP_RX: now also ESP-USART.1, ESP8266.URXD, STM_CHIP.16; no longer JP14.1, U$3.URXD, U1.53
- net ESP_TX: now also ESP-USART.2, ESP8266.UTXD, STM_CHIP.17; no longer JP14.2, U$3.UTXD, U1.54
- net ETH_CS: now also STM_CHIP.33; no longer R8.1, U1.20
- net ETH_MISO: now also STM_CHIP.35; no longer U1.22
- net ETH_MOSI: now also STM_CHIP.36; no longer U1.23
- net ETH_SCK: now also STM_CHIP.34; no longer U1.21
- net GESP: now also ESP-C1.2, ESP-GND.2, ESP-GPIO0.3, ESP8266.GND, ESP8266.GPIO15; no longer C54.2, JP12.2, JP13.3, U$3.GND, U$3.GPIO15
- net GEXT: now also ESP-GND.3, ESP-GND.4; no longer JP12.3
- net GND: no longer C40.2, C42.2, IC2.8, IC3.8, JP2.8, R25-10K.2, R28-10K.2, SV1.2, T1.E, T2.E, U$1.15, U$1.9, U$4.15, U$4.9
- net IBN: now also ADE-7.1, ADE-R9.1, CT2.5; no longer J2.1, R30.1
- net ICN: now also ADE-R10.1, ADE-R12.1, CT3.5; no longer J3.1, JP4.2, R31.1
- net LCD_CS: now also LCD_ILI9341.7, STM_CHIP.20; no longer JP2.7, U1.33
- net LCD_MISO: now also LCD_ILI9341.1, LCD_SD.3, STM_CHIP.22; no longer JP2.1, U1.35
- net LCD_MOSI: now also LCD_ILI9341.4, LCD_SD.2, STM_CHIP.23; no longer JP2.4, U1.36
- net LCD_SCK: now also LCD_ILI9341.3, LCD_SD.4, STM_CHIP.21; no longer JP2.3, U1.34
- net LINKLED: now also ETH-R5.1; no longer R20.1
- net N$1: now also STM-C5.2, STM-XTAL2.1, STM_CHIP.3; no longer C4.2, U1.3, Y1.1
- net N$11: now also ETH-R4.2, ETHERNET.10; no longer CN1.10, R19.2
- net N$12: now also ETH-R5.2, ETHERNET.11; no longer CN1.11, R20.2
- net N$13: now also SIM900-R1.1; no longer R9-22.1
- net N$14: now also SIM900-C4.1; no longer C10-4U7.1
- net N$15: now also SIM900-ANT.ANTENNA; no longer X1.ANTENNA
- net N$16: now also SIM900-LED1.A, SIM900-R4.1; no longer LED1.A, R20-1K.1
- net N$17: now also SIM900-LED1.C, SIM900-T1.C; no longer LED1.C, T1.C
- net N$18: now also SIM900-R5.1, SIM900-R6.1, SIM900-T1.B; no longer R23-1K.1, R25-10K.1, T1.B
- net N$19: now also SIM900-LED2.A, SIM900-R7.1; no longer LED2.A, R26-1K.1
- net N$2: now also STM-C6.1, STM-XTAL2.2, STM_CHIP.4; no longer C3.1, U1.4, Y1.2
- net N$20: now also SIM900-LED2.C, SIM900-T2.C; no longer LED2.C, T2.C
- net N$21: now also SIM900-R8.1, SIM900-R9.1, SIM900-T2.B; no longer R27-1K.1, R28-10K.1, T2.B
- net N$22: now also ETH-C2.1, ETHERNET.7; no longer C20.1, CN1.7
- net N$23: now also ETH-C1.2, ETH-R3.1, ETHERNET.3; no longer C18.2, CN1.3, R25.1
- net N$24: now also ADE-C7.1, ADER-11.2; no longer C25.1, R28.2
- net N$25: now also ADE-7.2, ADE-R8.1, CT2.1; no longer R23.1, R24.2
- net N$26: now also ETH-C4.1, ETHERNET.8; no longer C21.1, CN1.8
- net N$27: now also ADE-C3.1, ADE-R5.2; no longer C23.1, R26.2
- net N$28: now also ADE-C4.1, ADE-R6.2; no longer C26.1, R29.2
- net N$29: now also ETH-C3.2, ETH-R6.1, ETH-R7.2, ETHERNET.6; no longer C19.2, CN1.6
- net N$3: now also SIM900-R3.1; no longer R11-22.1
- net N$30: now also ADE-C6.1, ADE-R9.2; no longer C27.1, R30.2
- net N$31: now also ADE-C5.1, ADE-R8.2; no longer C24.1, R27.2
- net N$32: now also ADE-C10.1, ADE-C9.1; no longer C29.1, C30.1
- net N$33: now also ADE-C11.1, ADE-XTAL.1; no longer C32.1, Y3.1
- net N$34: now also ADE-C12.1, ADE-XTAL.2; no longer C31.1, Y3.2
- net N$35: now also ADE-C2.1, ADE-R3.2; no longer C33.1, R35.2
- net N$36: now also ADE-R1.1, VAC_IN.PWR; no longer C34.1, IC4.16, R32.2, R36.2
- net N$37: now also ADE-C1.1, ADE-R1.2, ADE-R2.2, IC4.14, IC4.16; no longer C35.1, R33.2, R37.2
- net N$38: now also W5500-C3.1; no longer C14.1
- net N$4: now also STM-C7.1, STM-R1.1, STM-S1.3, STM_CHIP.2; no longer C5.1, R2.1, S1.3, U1.2
- net N$40: now also ADE-C8.1, ADE-R12.2, IC4.10; no longer C36.1, IC4.14, R34.2, R38.2
- net N$41: now also W5500-C4.1; no longer C15.1
- net N$42: now also W5500-R11.2; no longer R6.2
- net N$43: now also W5500-HD1.2, W5500-R13.2; no longer JP7.2, R39.2
- net N$44: now also SIM900-R10.2, SIM900-T3.B; no longer R41.2, T9.B
- net N$45: now also SIM900-R11.2, SIM900-T4.B; no longer R42.2, T3.B
- net N$46: now also W5500-HD2.2, W5500-R12.2; no longer JP8.2, R40.2
- net N$49: now also W5500-C1.1, W5500-R10.1, W5500-XTAL.1; no longer C16.1, Q1.1, R9.1
- net N$5: now also STM-C7.2, STM-R2.2; no longer C5.2, R1.2
- net N$50: now also W5500-C2.1, W5500-R10.2, W5500-XTAL.2; no longer C17.1, Q1.2, R9.2
- net N$57: now also W5500-R8.1; no longer R14.1
- net N$58: now also W5500-R7.1; no longer R15.1
- net N$59: now also W5500-R6.1; no longer R16.1
- net N$6: now also STM-C2.2, STM-XTAL1.1, STM_CHIP.5; no longer C11.2, U1.5, Y2.1
- net N$60: now also W5500-R5.1; no longer R17.1
- net N$61: now also W5500-R4.1; no longer R18.1
- net N$62: now also W5500-R1.2; no longer R12.2
- net N$63: now also W5500-R2.2; no longer R11.2
- net N$64: now also W5500-R3.2; no longer R10.2
- net N$7: now also STM-C3.1, STM-XTAL1.2, STM_CHIP.6; no longer C10.1, U1.6, Y2.2
- net N$8: now also SIM900-R2.1; no longer R10-22.1
- net N$9: now also STM-C8.2, STM-R3.2; no longer C13.2, R3.2
- net NRST: now also STM-C8.1, STM-S2.3, STM_CHIP.7; no longer C13.1, S2.3, U1.7
- net Q1: now also SR_OUT1.1; no longer JP15.1
- net Q10: now also SR_OUT2.2; no longer JP16.2
- net Q11: now also SR_OUT2.3; no longer JP16.3
- net Q12: now also SR_OUT2.4; no longer JP16.4
- net Q13: now also SR_OUT2.5; no longer JP16.5
- net Q14: now also SR_OUT2.6; no longer JP16.6
- net Q15: now also SR_OUT2.7; no longer JP16.7
- net Q16: now also SR_OUT2.8; no longer JP16.8
- net Q2: now also SR_OUT1.2; no longer JP15.2
- net Q3: now also SR_OUT1.3; no longer JP15.3
- net Q4: now also SR_OUT1.4; no longer JP15.4
- net Q5: now also SR_OUT1.5; no longer JP15.5
- net Q6: now also SR_OUT1.6; no longer JP15.6
- net Q7: now also SR_OUT1.7; no longer JP15.7
- net Q8: now also SR_OUT1.8; no longer JP15.8
- net Q9: now also SR_OUT2.1; no longer JP16.1
- net RXN: now also ETH-C4.2, ETH-R7.1; no longer C21.2, R24.1
- net RXP: now also ETH-C2.2, ETH-R6.2; no longer C20.2, R23.2
- net SD_CS: now also LCD_SD.1, STM_CHIP.26; no longer JP3.1
- net SERIAL_RX: now also STM-USART.3, STM_CHIP.43; no longer JP9.3, U1.43
- net SERIAL_TX: now also STM-USART.2, STM_CHIP.42; no longer JP9.2, U1.42
- net SIM_NETLIGHT: now also SIM900-R8.2; no longer R27-1K.2
- net SIM_PWRKEY: now also SIM900-R10.1, STM_CHIP.61; no longer IC1.P$1, T9.C, U1.24
- net SIM_RESET: now also SIM900-R11.1, STM_CHIP.62; no longer IC1.P$16, T3.C, U1.25
- net SIM_RX: now also STM_CHIP.51; no longer U1.51
- net SIM_STATUS: now also SIM900-R5.2; no longer R23-1K.2
- net SIM_TX: now also STM_CHIP.52; no longer U1.52
- net SR_DS: now also STM_CHIP.11; no longer U1.8
- net SR_RST: now also STM_CHIP.8; no longer U1.11
- net SWO: now also STM-USART.4, STM_CHIP.55; no longer U1.55
- net TXN: now also ETH-R2.1, ETHERNET.2; no longer CN1.2, R22.1
- net TXP: now also ETH-R1.1, ETHERNET.1; no longer CN1.1, R21.1
- net USIM_CLK: now also SIM900-R2.2, SIM_HOLDER.3; no longer R10-22.2, U$2.3
- net USIM_DATA: now also SIM900-R3.2, SIM_HOLDER.4; no longer R11-22.2, U$2.4
- net USIM_RESET: now also SIM900-R1.2, SIM_HOLDER.2; no longer R9-22.2, U$2.2
- net USIM_VCC: now also SIM900-C5.1, SIM900-C6.1, SIM_C1.2, SIM_C2.2, SIM_HOLDER.1; no longer C11-22P.1, C9-100N.1, CSIM_100N.2, CSIM_22P.2, U$2.1
- net VCC: now also ETH-R1.2, ETH-R2.2, ETH-R3.2, STM-C9.1, STM-L1.2, STM_CHIP.13, SYS-C4.1, SYS-R2.2, W5500-C10.1, W5500-C11.1, W5500-C6.1, W5500-C7.1, W5500-C8.1, W5500-C9.1; no longer C1.1, C47.1, C48.1, C49.1, C50.1, C56.1, IC2.16, IC3.16, JP2.9, JP9.1, L1600R.2, R21.2, R22.2, R25.2, R43.2, SV1.8, U1.13
- net VDD: now also DCDC-3.5V.OUTP#1, DCDC-3.5V.OUTP#2, ESP-VDD.1, ETHERNET.12, ETHERNET.9, IC1.P$55, IC1.P$56, IC1.P$57, IC2.16, IC3.16, LCD-R1.2, LCD_ILI9341.9, SIM900-C1.+, SIM900-C2.+, SIM900-C3.+, SIM900-R4.2, SIM900-R7.2, STM-C1.2, STM-C10.1, STM-C11.1, STM-C12.1, STM-C13.1, STM-L1.1, STM-R1.2, STM-USART.1, STM_CHIP.1, STM_CHIP.19, STM_CHIP.32, STM_CHIP.48, STM_CHIP.64, SYS-C3.1, SYS-R2.1, W5500-C5.1, W5500-HD1.1, W5500-HD2.1, W5500-R1.1, W5500-R2.1, W5500-R3.1, W5500-R9.2; no longer C12.2, C46.+, C53.1, C55.1, C6.1, C7.1, C8.1, C9.1, CN1.12, CN1.9, D4.A, IC6.2, JP1.1, JP7.1, JP8.1, L1600R.1, R10.1, R11.1, R12.1, R13.2, R2.2, R43.1, R7.2, R8.2, U1.1, U1.19, U1.32, U1.48, U1.64
- net VESP: now also ESP-C1.1, ESP-GPIO0.1, ESP-VDD.2, ESP8266.CH_PD, ESP8266.GPIO2, ESP8266.VCC; no longer C54.1, JP1.2, JP13.1, U$3.CH_PD, U$3.GPIO2, U$3.VCC
- net VEXT: now also ESP-VDD.3, ESP-VDD.4; no longer JP1.3
Routing:
- net DGND: track 3.07 -> 34.7 mm, vias 0 -> 3
- net Q8: track 0.00 -> 30.0 mm, vias 0 -> 2
- net Q16: track 0.00 -> 28.7 mm, vias 0 -> 2
- net Q2: track 0.00 -> 27.8 mm, vias 0 -> 1
- net Q10: track 0.00 -> 27.6 mm, vias 0 -> 1
- net Q1: track 0.00 -> 27.5 mm, vias 0 -> 1
- net Q9: track 0.00 -> 26.3 mm, vias 0 -> 1
- net Q6: track 0.00 -> 25.2 mm, vias 0 -> 2
- net Q14: track 0.00 -> 24.4 mm, vias 0 -> 2
- net Q12: track 0.00 -> 23.1 mm, vias 0 -> 1
- net Q4: track 0.00 -> 22.8 mm, vias 0 -> 1
- net Q11: track 0.00 -> 14.7 mm, vias 0 -> 2
- net Q3: track 0.00 -> 14.1 mm, vias 0 -> 2
- net Q7: track 0.00 -> 11.9 mm, vias 0 -> 2
- net Q15: track 0.00 -> 11.6 mm, vias 0 -> 2
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Other:
- outline, holes or cut-outs redrawn
