File: eagle/EmonMbed.sch (EAGLE design)
At the start: 171 parts, among them IC2 74HC595D, IC3 74HC595D, IC4 ADE7758RW, IC6 REG1117, IC7 7805DT, J1 CON_TERMINAL_BLOCK_02-5MM, J2 CON_TERMINAL_BLOCK_02-5MM, J3 CON_TERMINAL_BLOCK_02-5MM, J4 CON_TERMINAL_BLOCK_03-5MM, J7 CON_TERMINAL_BLOCK_02-5MM, Q1 25MHz, U1 STM32L152RBT6, U2 W5500, Y1 32.768kHz, Y2 32.768kHz

Commit message: Updated Final Schematics
Parts:
- removed C10-4U7, C11-22P, C9-100N: (no value), rcl:C-EUC0603
- removed C2: 4.7uF, rcl:C-EUC0603
- removed C22: 1nF, rcl:C-EUC0603
- removed C23, C34, C35, C36: 33nF, SparkFun-Passives:CAP0603-CAP
- removed C37: 10uF, rcl:CPOL-USC/6032-28R
- removed C38, C39, C40, C41, C42, C43, C44, C55, C56: 0.1uF, rcl:C-USC0805
- removed C45, C59: 10uF, rcl:CPOL-US153CLV-0605
- removed C46, C60: 0.1uF, rcl:CPOL-US153CLV-0605
- removed C54: 100nF, rcl:C-EUC0603
- removed C7-100U: 100uF, rcl:CPOL-EU153CLV-0605
- removed C8-100U: (no value), rcl:CPOL-EU153CLV-0605
- removed D1, D2, D3, D4: 1N4001, diode:DIODE-DO-214AC
- removed IC6: REG1117, burr-brown:REG1117
- removed IC7: 7805DT, linear:7805DT
- removed J1, J2, J3, J7: CON_TERMINAL_BLOCK_02-5MM, dp_devices:CON_TERMINAL_BLOCK_02-5MM
- removed J4: CON_TERMINAL_BLOCK_03-5MM, dp_devices:CON_TERMINAL_BLOCK_03-5MM
- removed JP1: Vsel, pinhead:PINHD-1X3
- removed JP12: (no value), pinhead:PINHD-1X3
- removed JP15, JP16: (no value), pinhead:PINHD-2X5/90
- removed JP2: TFT LCD ILI9341, pinhead:PINHD-1X9
- removed JP3: SD CARD TFT LCD, pinhead:PINHD-1X4
- removed JP4, JP5, JP6: (no value), jumper:JP1E
- removed JP9: USART, pinhead:PINHD-1X4
- removed L1: 150Mhz, rcl:L-USWE-TPC
- removed LED1, LED2: (no value), microbuilder:LED0805_NOOUTLINE
- removed R10-22, R11-22, R20-1K, R23-1K, R25-10K, R26-1K, R27-1K, R28-10K, R9-22: (no value), rcl:R-EU_R0603
- removed R19: 330, resistor:R-US_R0603
- removed R26, R36, R37, R38: 1K, SparkFun-Passives:RESISTOR0603-RES
- removed R32, R33, R34: 1M, SparkFun-Passives:RESISTOR0603-RES
- removed R4, R43: 10, SparkFun-Passives:RESISTOR0603-RES
- removed R41, R42: R120, resistor:R-EU_R0603
- removed R5: 12.4k, resistor:R-US_R0603
- removed R7, R8: 10k, resistor:R-US_R0603
- removed SV1: (no value), con-lstb:MA08-1
- removed T1, T2: (no value), transistor:MMBT2222ALT1-NPN-SOT23-BEC
- removed T3, T9: (no value), transistor-neu-to92:MMBT2222ALT1-NPN-SOT23-BEC
- removed U$1, U$4: ADUM1402, adum140x:ADUM1402
- removed X1: (no value), microbuilder:SMACONNECTOR
- removed X2: (no value), con-ptr500:AK500/2-H
- added ADE-7, ADE-R10, ADE-R4: 33R, SparkFun-Passives:RESISTOR0603-RES
- added ADE-C1, ADE-C3: 33nF, SparkFun-Passives:CAP0603-CAP
- added ADE-C13: 10uF, rcl:CPOL-USC/6032-28R
- added ADE-C14, SYS-C1, SYS-C2, SYS-C3, SYS-C4: 0.1uF, rcl:C-USC0805
- added ADE-R1: 81K, SparkFun-Passives:RESISTOR0603-RES
- added ADE-R2, ADE-R5: 1K, SparkFun-Passives:RESISTOR0603-RES
- added CT1, CT2, CT3: 100A, microbuilder:AUDIO_STEREOJACK
- added ESP-C1, SIM900-C5: 100nF, rcl:C-EUC0603
- added ESP-GND, LCD_SD: (no value), pinhead:PINHD-1X4
- added ESP-VDD: Vsel, pinhead:PINHD-1X4
- added ETH-R4: 330, resistor:R-US_R0603
- added J5: POWER_JACKPTH, SparkFun-Connectors:POWER_JACKPTH
- added LCD-R1: 680R, SparkFun-Passives:RESISTOR0603-RES
- added LCD_ILI9341: (no value), pinhead:PINHD-1X9
- added SIM900-ANT: (no value), microbuilder:SMACONNECTOR
- added SIM900-C1, SIM900-C2, SIM900-C3: 100uF, rcl:CPOL-EU153CLV-0605
- added SIM900-C4: 4u7, rcl:C-EUC0603
- added SIM900-C6: 22pF, rcl:C-EUC0603
- added SIM900-LED1, SIM900-LED2: (no value), microbuilder:LED0805_NOOUTLINE
- added SIM900-R1, SIM900-R2, SIM900-R3: 22R, rcl:R-EU_R0603
- added SIM900-R10, SIM900-R11: 120R, resistor:R-EU_R0603
- added SIM900-R4, SIM900-R7: 680R, rcl:R-EU_R0603
- added SIM900-R5, SIM900-R8: 1K, rcl:R-EU_R0603
- added SIM900-R6, SIM900-R9: 10K, rcl:R-EU_R0603
- added SIM900-T1, SIM900-T2: (no value), transistor:MMBT2222ALT1-NPN-SOT23-BEC
- added SIM900-T3, SIM900-T4: (no value), transistor-neu-to92:MMBT2222ALT1-NPN-SOT23-BEC
- added SR_OUT1, SR_OUT2: (no value), pinhead:PINHD-2X4/90
- added STM-USART: USART, pinhead:PINHD-1X5
- added SYS-L1: 150Mhz, rcl:L-USWE-TPC
- added SYS-R1, SYS-R2: 10R, SparkFun-Passives:RESISTOR0603-RES
- added VAC_IN: 9V, SparkFun-Connectors:POWER_JACKPTH
- ADE-XTAL: value (none) -> 10MHz
- IC1: value (none) -> SIM900
- SIM_C1: value (none) -> 100nF
- SIM_C2: value (none) -> 22pF
- STM_CHIP: value STM32L152RBT6 -> STM32F103RBT6
- renumbered C1 to STM-C9, C10 to STM-C3, C11 to STM-C2, C12 to STM-C1, C13 to STM-C8, C14 to W5500-C3, C15 to W5500-C4, C16 to W5500-C1, C17 to W5500-C2, C18 to ETH-C1, C19 to ETH-C3, C20 to ETH-C2, C21 to ETH-C4, C24 to ADE-C5, C25 to ADE-C7, C26 to ADE-C4, C27 to ADE-C6, C28 to ADE-C8, C29 to ADE-C9, C3 to STM-C6, C30 to ADE-C10, C31 to ADE-C12, C32 to ADE-C11, C33 to ADE-C2, C4 to STM-C5, C47 to W5500-C6, C48 to W5500-C7, C49 to W5500-C8, C5 to STM-C7, C50 to W5500-C9, C51 to W5500-C10, C52 to W5500-C11, C53 to W5500-C5, C6 to STM-C10, C7 to STM-C11, C8 to STM-C12, C9 to STM-C13, CN1 to ETHERNET, CSIM_100N to SIM_C1, CSIM_22P to SIM_C2, JP13 to ESP-GPIO0, JP14 to ESP-USART, JP7 to W5500-HD1, JP8 to W5500-HD2, L1600R to STM-L1, Q1 to W5500-XTAL, R1 to STM-R2, R10 to W5500-R3, R11 to W5500-R2, R12 to W5500-R1, R13 to W5500-R9, R14 to W5500-R8, R15 to W5500-R7, R16 to W5500-R6, R17 to W5500-R5, R18 to W5500-R4, R2 to STM-R1, R20 to ETH-R5, R21 to ETH-R1, R22 to ETH-R2, R23 to ETH-R6, R24 to ETH-R7, R25 to ETH-R3, R27 to ADE-R8, R28 to ADER-11, R29 to ADE-R6, R3 to STM-R3, R30 to ADE-R9, R31 to ADE-R12, R35 to ADE-R3, R39 to W5500-R13, R40 to W5500-R12, R6 to W5500-R11, R9 to W5500-R10, S1 to STM-S1, S2 to STM-S2, U$2 to SIM_HOLDER, U$3 to ESP8266, U$6 to DCDC-3.5V, U1 to STM_CHIP, Y1 to STM-XTAL2, Y2 to STM-XTAL1, Y3 to ADE-XTAL
Connections:
- removed net !ADECS: IC4.DIF.CS, U$4.VOC
- removed net !CS: SV1.3
- removed net ADEAPCF: IC4.CAL.APCF, U$1.VIA
- removed net ADEIN: IC4.DIF.DI, U$1.VOD
- removed net ADEIRQ: IC4.DIF.IRQ, U$4.VIB
- removed net ADEOUT: IC4.DIF.DO, U$1.VIB
- removed net ADESCK: IC4.DIF.SCK, U$1.VOC
- removed net ADEVARCF: IC4.CAL.VARCF, U$4.VIA
- removed net APCF: STM_CHIP.PB4, U$1.VOA
- removed net AVADE: C44.1, IC4.PWR.AVDD, R4.2
- removed net D/C: JP2.5
- removed net DGND1: W5500-C10.2, W5500-C11.2
- removed net DS_OE: IC2A.G, IC3A.G
- removed net EXRES1: R5.2, U2.EXRES1
- removed net GND: C40.2, C42.2, JP2.8, R25-10K.2, R28-10K.2, SV1.2, T1.E, T2.E, U$1.GND2@1, U$1.GND2@2, U$4.GND2@1, U$4.GND2@2
- removed net I2C_SCL: STM_CHIP.PB8
- removed net I2C_SDA: STM_CHIP.PB9
- removed net IAN: ADE-R6.1, J1.1
- removed net IAP: J1.2, R26.1
- removed net IBP: ADE-R8.1, J2.2
- removed net ICP: ADER-11.1, J3.2, JP5.2
- removed net INTN: R7.1, U2.INT_N
- removed net IRQ: STM_CHIP.PB6, SV1.7, U$4.VOA
- removed net LED: JP2.2
- removed net MISO: SV1.6
- removed net MOSI: SV1.4
- removed net N$40 (its old number): C36.1, IC4.U.VCP, R34.2, R38.2
- removed net PB10: STM_CHIP.PB10
- removed net PB11: C2.1, STM_CHIP.PB11
- removed net PWRKEY: R41.1
- removed net RESET: JP2.6, R42.1
- removed net RSTN: U2.RST_N, W5500-R9.1
- removed net SCK: SV1.5
- removed net SD_MISO: JP3.3
- removed net SD_MOSI: JP3.2
- removed net SD_SCK: JP3.4
- removed net SHCP: IC2A.SCK, IC3A.SCK, STM_CHIP.PC2
- removed net STCP: IC2A.RCK, IC3A.RCK, STM_CHIP.PC1
- removed net VADE: C37.+, C38.1, C39.1, C40.1, C41.1, C42.1, C43.1, C60.+, D3.A, IC4.PWR.DVDD, IC7.VO, R4.1, U$1.VDD1, U$1.VDD2, U$1.VE1, U$1.VE2, U$4.VDD1, U$4.VDD2, U$4.VE1, U$4.VE2
- removed net VAP: J4.1, R32.1
- removed net VARCF: STM_CHIP.PB5, U$4.VOB
- removed net VBP: J4.2, R33.1
- removed net VCC1: W5500-C10.1, W5500-C11.1
- removed net VCP: J4.3, JP6.2, R34.1
- removed net VIN: C45.+, C59.+, D1.C, D2.C, D3.C, D4.C, DCDC-3.5V.VIN, IC6.VIN, IC7.VI
- removed net VN: ADE-R3.1, J7.1, J7.2
- removed net VRAW: D1.A, D2.A, X2-1.KL
- removed net VSIM: C7-100U.+, C8-100U.+, DCDC-3.5V.VOUT, IC1.VBAT1, IC1.VBAT2, IC1.VBAT3
- new net ADE_APCF: IC4.CAL.APCF, STM_CHIP.PB5
- new net ADE_IRQ: IC4.DIF.IRQ, STM_CHIP.PB7
- new net ADE_VARCF: IC4.CAL.VARCF, STM_CHIP.PB6
- new net AVDD: IC4.PWR.AVDD, SYS-C2.1, SYS-R1.2
- new net ETH_RSTN: STM_CHIP.PC6, U2.RST_N, W5500-R9.1
- new net LCD_D/C: LCD_ILI9341.5, STM_CHIP.PC4
- new net LCD_LED: LCD-R1.1, LCD_ILI9341.2
- new net LCD_RESET: LCD_ILI9341.6, STM_CHIP.PC5
- new net N$39: ADE-R4.2, ADE-R5.1, CT1.1
- new net N$47: ADE-R4.1, ADE-R6.1, CT1.5
- new net N$48: ADE-R10.2, ADER-11.1, CT3.1
- new net N$51: ADE-R3.1, VAC_IN.GND, VAC_IN.GNDBREAK
- new net SIM900_PWRKEY: IC1.PWRKEY, SIM900-T3.C
- new net SIM900_RESET: IC1.NRESET, SIM900-T4.C
- new net SR_SHCP: IC2A.SCK, IC3A.SCK, STM_CHIP.PC1
- new net SR_STCP: IC2A.RCK, IC3A.RCK, STM_CHIP.PC2
- net +5V: now also ADE-C13.+, ADE-C14.1, DCDC-3.5V.VIN, IC4.PWR.DVDD, J5.PWR, SYS-C1.1, SYS-R1.1; no longer R20-1K.2, R26-1K.2
- net ACTLED: now also ETH-R4.1; no longer R19.1
- net ADE_CS: now also IC4.DIF.CS, STM_CHIP.PA15; no longer STM_CHIP.PA12, U$4.VIC
- net ADE_MISO: now also IC4.DIF.DO, STM_CHIP.PA12; no longer STM_CHIP.PA14, U$1.VOB
- net ADE_MOSI: now also IC4.DIF.DI, STM_CHIP.PA13; no longer STM_CHIP.PA15, U$1.VID
- net ADE_SCK: now also IC4.DIF.SCK, STM_CHIP.PA14; no longer STM_CHIP.PA13, U$1.VIC
- net AGND: now also ADE-C1.2, ADE-C3.2, ADE-R2.1, SYS-C2.2, SYS-C4.2, SYS-L1.1, W5500-C10.2, W5500-C11.2; no longer C22.1, C23.2, C34.2, C35.2, C36.2, C44.2, C56.2, JP4.1, JP5.1, JP6.1, L1.1, R36.1, R37.1, R38.1
- net DGND: now also ADE-C13.-, ADE-C14.2, ESP-GND.1, IC2A.G, IC2P.GND, IC3A.G, IC3P.GND, J5.GND, J5.GNDBREAK, LCD_ILI9341.8, SIM900-ANT.GND1, SIM900-ANT.GND2, SIM900-ANT.GND3, SIM900-ANT.GND4, SIM900-C1.-, SIM900-C2.-, SIM900-C3.-, SIM900-C4.2, SIM900-C5.2, SIM900-C6.2, SIM900-R6.2, SIM900-R9.2, SIM900-T1.E, SIM900-T2.E, SIM900-T3.E, SIM900-T4.E, STM-USART.5, SYS-C1.2, SYS-C3.2, SYS-L1.2; no longer C10-4U7.2, C11-22P.2, C2.2, C22.2, C37.-, C38.2, C39.2, C41.2, C43.2, C45.-, C46.-, C55.2, C59.-, C60.-, C7-100U.-, C8-100U.-, C9-100N.2, IC6.GND, IC7.GND, JP12.1, JP9.4, L1.2, R5.1, T3.E, T9.E, U$1.GND1@1, U$1.GND1@2, U$4.GND1@1, U$4.GND1@2, X1.GND1, X1.GND2, X1.GND3, X1.GND4, X2-2.KL
- net ESP_RX: now also STM_CHIP.PA2; no longer STM_CHIP.PC12
- net ESP_TX: now also STM_CHIP.PA3; no longer STM_CHIP.PD2
- net ETH_CS: now also STM_CHIP.PB12; no longer R8.1, STM_CHIP.PA4
- net ETH_MISO: now also STM_CHIP.PB14; no longer STM_CHIP.PA6
- net ETH_MOSI: now also STM_CHIP.PB15; no longer STM_CHIP.PA7
- net ETH_SCK: now also STM_CHIP.PB13; no longer STM_CHIP.PA5
- net GESP: now also ESP-C1.2, ESP-GND.2; no longer C54.2, JP12.2
- net GEXT: now also ESP-GND.3, ESP-GND.4; no longer JP12.3
- net IBN: now also ADE-7.1, CT2.5; no longer J2.1
- net ICN: now also ADE-R10.1, CT3.5; no longer J3.1, JP4.2
- net LCD_CS: now also LCD_ILI9341.7, STM_CHIP.PA4; no longer JP2.7, STM_CHIP.PB12
- net LCD_MISO: now also LCD_ILI9341.1, LCD_SD.3, STM_CHIP.PA6; no longer JP2.1, STM_CHIP.PB14
- net LCD_MOSI: now also LCD_ILI9341.4, LCD_SD.2, STM_CHIP.PA7; no longer JP2.4, STM_CHIP.PB15
- net LCD_SCK: now also LCD_ILI9341.3, LCD_SD.4, STM_CHIP.PA5; no longer JP2.3, STM_CHIP.PB13
- net N$11: now also ETH-R4.2; no longer R19.2
- net N$13: now also SIM900-R1.1; no longer R9-22.1
- net N$14: now also SIM900-C4.1; no longer C10-4U7.1
- net N$15: now also SIM900-ANT.ANT; no longer X1.ANT
- net N$16: now also SIM900-LED1.A, SIM900-R4.1; no longer LED1.A, R20-1K.1
- net N$17: now also SIM900-LED1.C, SIM900-T1.C; no longer LED1.C, T1.C
- net N$18: now also SIM900-R5.1, SIM900-R6.1, SIM900-T1.B; no longer R23-1K.1, R25-10K.1, T1.B
- net N$19: now also SIM900-LED2.A, SIM900-R7.1; no longer LED2.A, R26-1K.1
- net N$20: now also SIM900-LED2.C, SIM900-T2.C; no longer LED2.C, T2.C
- net N$21: now also SIM900-R8.1, SIM900-R9.1, SIM900-T2.B; no longer R27-1K.1, R28-10K.1, T2.B
- net N$25: now also ADE-7.2, ADE-R8.1, CT2.1; no longer ETH-R6.1, ETH-R7.2
- net N$27: now also ADE-C3.1, ADE-R5.2; no longer C23.1, R26.2
- net N$29: now also ETH-R6.1, ETH-R7.2
- net N$3: now also SIM900-R3.1; no longer R11-22.1
- net N$36: now also ADE-R1.1, VAC_IN.PWR; no longer C34.1, IC4.U.VAP, R32.2, R36.2
- net N$37: now also ADE-C1.1, ADE-R1.2, ADE-R2.2, IC4.U.VAP, IC4.U.VCP; no longer C35.1, R33.2, R37.2
- net N$44: now also SIM900-R10.2, SIM900-T3.B; no longer R41.2, T9.B
- net N$45: now also SIM900-R11.2, SIM900-T4.B; no longer R42.2, T3.B
- net N$8: now also SIM900-R2.1; no longer R10-22.1
- net Q1: now also SR_OUT1.1; no longer JP15.1
- net Q10: now also SR_OUT2.2; no longer JP16.2
- net Q11: now also SR_OUT2.3; no longer JP16.3
- net Q12: now also SR_OUT2.4; no longer JP16.4
- net Q13: now also SR_OUT2.5; no longer JP16.5
- net Q14: now also SR_OUT2.6; no longer JP16.6
- net Q15: now also SR_OUT2.7; no longer JP16.7
- net Q16: now also SR_OUT2.8; no longer JP16.8
- net Q2: now also SR_OUT1.2; no longer JP15.2
- net Q3: now also SR_OUT1.3; no longer JP15.3
- net Q4: now also SR_OUT1.4; no longer JP15.4
- net Q5: now also SR_OUT1.5; no longer JP15.5
- net Q6: now also SR_OUT1.6; no longer JP15.6
- net Q7: now also SR_OUT1.7; no longer JP15.7
- net Q8: now also SR_OUT1.8; no longer JP15.8
- net Q9: now also SR_OUT2.1; no longer JP16.1
- net SD_CS: now also LCD_SD.1, STM_CHIP.PB0; no longer JP3.1
- net SERIAL_RX: now also STM-USART.3; no longer JP9.3
- net SERIAL_TX: now also STM-USART.2; no longer JP9.2
- net SIM_NETLIGHT: now also SIM900-R8.2; no longer R27-1K.2
- net SIM_PWRKEY: now also SIM900-R10.1, STM_CHIP.PB8; no longer IC1.PWRKEY, STM_CHIP.PC4, T9.C
- net SIM_RESET: now also SIM900-R11.1, STM_CHIP.PB9; no longer IC1.NRESET, STM_CHIP.PC5, T3.C
- net SIM_STATUS: now also SIM900-R5.2; no longer R23-1K.2
- net SR_DS: now also STM_CHIP.PC3; no longer STM_CHIP.PC0
- net SR_RST: now also STM_CHIP.PC0; no longer STM_CHIP.PC3
- net SWO: now also STM-USART.4
- net USIM_CLK: now also SIM900-R2.2; no longer R10-22.2
- net USIM_DATA: now also SIM900-R3.2; no longer R11-22.2
- net USIM_RESET: now also SIM900-R1.2; no longer R9-22.2
- net USIM_VCC: now also SIM900-C5.1, SIM900-C6.1; no longer C11-22P.1, C9-100N.1
- net VCC: now also SYS-C4.1, SYS-R2.2, W5500-C10.1, W5500-C11.1; no longer C56.1, JP2.9, JP9.1, R43.2, SV1.8
- net VDD: now also DCDC-3.5V.VOUT, ESP-VDD.1, IC1.VBAT1, IC1.VBAT2, IC1.VBAT3, IC2P.VCC, IC3P.VCC, LCD-R1.2, LCD_ILI9341.9, SIM900-C1.+, SIM900-C2.+, SIM900-C3.+, SIM900-R4.2, SIM900-R7.2, STM-USART.1, SYS-C3.1, SYS-R2.1; no longer C46.+, C55.1, D4.A, IC6.VOUT, JP1.1, R43.1, R7.2, R8.2
- net VESP: now also ESP-C1.1, ESP-VDD.2; no longer C54.1, JP1.2
- net VEXT: now also ESP-VDD.3, ESP-VDD.4; no longer JP1.3
Other:
- note removed: "LMS8117A"
- moved on the sheet: IC1, IC3
